Commit message: Fixed Launch and URDF files for noetic support

File: urdf/2r_description.xacro (robot description, xacro)
@@ -6,19 +6,22 @@
   LABORATORIO / ROBOTICA 2020-1
   PROF: PEDRO CARDENAS
-  URDF ROBOT DESCRITION EXAMPLE FOR GAZEBO SIMULATION
-  AUTHOR: JURGEN KREJCI MUNOZ
+  URDF ROBOT DESCRIPTION EXAMPLE FOR GAZEBO SIMULATION
+  AUTHOR: JURGEN H. KREJCI MUNOZ
   ROBOT: 2R
+  MAIL: jhkrejcim@unal.edu.co
   VERSION: 1.0
+  TESTED ON ROS NOETIC (UBUNTU 20.04.1 LTS)
+  https://github.com/JurgenHK/2R-Manipulator-URDF
   -->
 <robot name="2R" xmlns:xacro="http://www.ros.org/wiki/xacro">
   <!-- Include -->
-  <xacro:include filename="$(find 2R_Gazebo)/urdf/links_joints.xacro" />
-  <xacro:include filename="$(find 2R_Gazebo)/urdf/robot_parameters.xacro" />
+  <xacro:include filename="$(find basic_2r_gazebo)/urdf/links_joints.xacro" />
+  <xacro:include filename="$(find basic_2r_gazebo)/urdf/robot_parameters.xacro" />
   <!-- END - Include -->
   <!-- Robot description -->
-  <m_link_mesh name="${link_00_name}"
+  <xacro:m_link_mesh name="${link_00_name}"
     origin_xyz="0 0 0"
     origin_rpy="0 0 0"
-    meshfile="package://2R_Gazebo/CAD/Base.dae"
+    meshfile="package://basic_2r_gazebo/CAD/Base.dae"
     mass="0.00272"
     ixx="0.00000006" ixy="0" ixz="0"
@@ -26,5 +29,5 @@
     izz="0.00000008"
   />
-  <m_joint name="${joint_01_name}"
+  <xacro:m_joint name="${joint_01_name}"
     type="revolute"
     axis_xyz="0 0 1"
@@ -33,8 +36,8 @@
     limit_e="100" limit_l="-3.14" limit_u="3.14" limit_v="0.5"
   />
-  <m_link_mesh name="${link_01_name}"
+  <xacro:m_link_mesh name="${link_01_name}"
     origin_xyz="0 0 0"
     origin_rpy="0 0 0"
-    meshfile="package://2R_Gazebo/CAD/Link1.dae"
+    meshfile="package://basic_2r_gazebo/CAD/Link1.dae"
     mass="0.002268"
     ixx="0.0000000181" ixy="0" ixz="0"
@@ -42,5 +45,5 @@
     izz="0.000000127"
   />
-  <m_joint name="${joint_02_name}"
+  <xacro:m_joint name="${joint_02_name}"
     type="revolute"
     axis_xyz="0 0 1"
@@ -49,8 +52,8 @@
     limit_e="100" limit_l="-3.14" limit_u="3.14" limit_v="0.5"
   />
-  <m_link_mesh name="${link_02_name}"
+  <xacro:m_link_mesh name="${link_02_name}"
     origin_xyz="0 0 0"
     origin_rpy="0 0 0"
-    meshfile="package://2R_Gazebo/CAD/Link2.dae"
+    meshfile="package://basic_2r_gazebo/CAD/Link2.dae"
     mass="0.002268"
     ixx="0.0000000181" ixy="0" ixz="0"
@@ -58,5 +61,5 @@
     izz="0.000000127"
   />
-  <m_joint name="${joint_03_name}"
+  <xacro:m_joint name="${joint_03_name}"
     type="prismatic"
     axis_xyz="0 0 1"
@@ -65,8 +68,8 @@
     limit_e="100" limit_l="0" limit_u="2" limit_v="0.5"
   />
-  <m_link_mesh name="${link_03_name}"
+  <xacro:m_link_mesh name="${link_03_name}"
     origin_xyz="0 0 0"
     origin_rpy="0 0 0"
-    meshfile="package://2R_Gazebo/CAD/Finger.dae"
+    meshfile="package://basic_2r_gazebo/CAD/Finger.dae"
     mass="0.002268"
     ixx="0.0000000181" ixy="0" ixz="0"
@@ -74,5 +77,5 @@
     izz="0.000000127"
   />
-  <m_joint_mimic name="${joint_04_name}"
+  <xacro:m_joint_mimic name="${joint_04_name}"
     type="prismatic"
     axis_xyz="0 0 1"
@@ -82,8 +85,8 @@
     mimic_joint="${joint_03_name}" m_multiplier="1" m_offset="0"
   />
-  <m_link_mesh name="${link_04_name}"
+  <xacro:m_link_mesh name="${link_04_name}"
     origin_xyz="0 0 0"
     origin_rpy="0 0 0"
-    meshfile="package://2R_Gazebo/CAD/Finger.dae"
+    meshfile="package://basic_2r_gazebo/CAD/Finger.dae"
     mass="0.002268"
     ixx="0.0000000181" ixy="0" ixz="0"
@@ -91,5 +94,5 @@
     izz="0.000000127"
   />
-  <create_noa name="NOA"
+  <xacro:create_noa name="NOA"
     origin_xyz="20 0 0"
     origin_rpy="-1.57 0 -1.57"

File: urdf/2r_description_gazebo.xacro (robot description, xacro)
@@ -6,14 +6,16 @@
   LABORATORIO / ROBOTICA 2020-1
   PROF: PEDRO CARDENAS
-  URDF ROBOT DESCRITION EXAMPLE FOR GAZEBO SIMULATION
-  AUTHOR: JURGEN KREJCI MUNOZ
+  URDF ROBOT DESCRIPTION EXAMPLE FOR GAZEBO SIMULATION
+  AUTHOR: JURGEN H. KREJCI MUNOZ
+  ROBOT: 2R
   MAIL: jhkrejcim@unal.edu.co
-  ROBOT: 2R
   VERSION: 1.0
+  TESTED ON ROS NOETIC (UBUNTU 20.04.1 LTS)
+  https://github.com/JurgenHK/2R-Manipulator-URDF
   -->
 <robot name="2R" xmlns:xacro="http://www.ros.org/wiki/xacro">
   <!-- Include-->
-  <xacro:include filename="$(find 2R_Gazebo)/urdf/links_joints.xacro" />
-  <xacro:include filename="$(find 2R_Gazebo)/urdf/robot_parameters.xacro" />
+  <xacro:include filename="$(find basic_basic_2r_gazebo)/urdf/links_joints.xacro" />
+  <xacro:include filename="$(find basic_basic_2r_gazebo)/urdf/robot_parameters.xacro" />
   <!-- END - Include -->
   <!-- Robot description -->
@@ -23,8 +25,8 @@
     <child link="${link_00_name}"/>
   </joint>
-  <m_link_mesh name="${link_00_name}"
+  <xacro:m_link_mesh name="${link_00_name}"
     origin_xyz="0 0 0"
     origin_rpy="0 0 0"
-    meshfile="package://2R_Gazebo/CAD/Base.stl"
+    meshfile="package://basic_2r_gazebo/CAD/Base.stl"
     mass="1.024"
     ixx="170.0" ixy="0" ixz="0"
@@ -32,5 +34,5 @@
     izz="170.0"
   />
-  <m_joint name="${joint_01_name}"
+  <xacro:m_joint name="${joint_01_name}"
     type="revolute"
     axis_xyz="0 0 1"
@@ -39,8 +41,8 @@
     limit_e="100" limit_l="-3.14" limit_u="3.14" limit_v="0.5"
   />
-  <m_link_mesh name="${link_01_name}"
+  <xacro:m_link_mesh name="${link_01_name}"
     origin_xyz="0 0 0"
     origin_rpy="0 0 0"
-    meshfile="package://2R_Gazebo/CAD/Link1.stl"
+    meshfile="package://basic_2r_gazebo/CAD/Link1.stl"
     mass="1.570"
     ixx="130.0" ixy="0" ixz="0"
@@ -48,5 +50,5 @@
     izz="90.0"
   />
-  <m_joint name="${joint_02_name}"
+  <xacro:m_joint name="${joint_02_name}"
     type="revolute"
     axis_xyz="0 0 1"
@@ -55,8 +57,8 @@
     limit_e="100" limit_l="-3.14" limit_u="3.14" limit_v="0.5"
   />
-  <m_link_mesh name="${link_02_name}"
+  <xacro:m_link_mesh name="${link_02_name}"
     origin_xyz="0 0 0"
     origin_rpy="0 0 0"
-    meshfile="package://2R_Gazebo/CAD/Link2.stl"
+    meshfile="package://basic_2r_gazebo/CAD/Link2.stl"
     mass="0.057"
     ixx="12.0" ixy="0" ixz="0"
@@ -64,5 +66,5 @@
     izz="12.0"
   />
-  <m_joint name="${joint_03_name}"
+  <xacro:m_joint name="${joint_03_name}"
     type="prismatic"
     axis_xyz="0 0 1"
@@ -71,8 +73,8 @@
     limit_e="100" limit_l="0" limit_u="2" limit_v="0.5"
   />
-  <m_link_mesh name="${link_03_name}"
+  <xacro:m_link_mesh name="${link_03_name}"
     origin_xyz="0 0 0"
     origin_rpy="0 0 0"
-    meshfile="package://2R_Gazebo/CAD/Finger.stl"
+    meshfile="package://basic_2r_gazebo/CAD/Finger.stl"
     mass="0.018"
     ixx="0.5" ixy="0" ixz="0"
@@ -80,5 +82,5 @@
     izz="0.5"
   />
-  <m_joint_mimic name="${joint_04_name}"
+  <xacro:m_joint_mimic name="${joint_04_name}"
     type="prismatic"
     axis_xyz="0 0 1"
@@ -88,8 +90,8 @@
     mimic_joint="${joint_03_name}" m_multiplier="1" m_offset="0"
   />
-  <m_link_mesh name="${link_04_name}"
+  <xacro:m_link_mesh name="${link_04_name}"
     origin_xyz="0 0 0"
     origin_rpy="0 0 0"
-    meshfile="package://2R_Gazebo/CAD/Finger.stl"
+    meshfile="package://basic_2r_gazebo/CAD/Finger.stl"
     mass="0.018"
     ixx="0.5" ixy="0" ixz="0"

File: urdf/links_joints.xacro (robot description, xacro)
@@ -6,8 +6,11 @@
   LABORATORIO / ROBOTICA 2020-1
   PROF: PEDRO CARDENAS
-  MACROS FOR LINKS AND JOINTS - ROBOT DESCRITION
-  AUTHOR: JURGEN KREJCI MUNOZ
+  URDF ROBOT DESCRIPTION EXAMPLE FOR GAZEBO SIMULATION
+  AUTHOR: JURGEN H. KREJCI MUNOZ
+  ROBOT: 2R
   MAIL: jhkrejcim@unal.edu.co
   VERSION: 1.0
+  TESTED ON ROS NOETIC (UBUNTU 20.04.1 LTS)
+  https://github.com/JurgenHK/2R-Manipulator-URDF
   -->
 <robot xmlns:xacro="http://www.ros.org/wiki/xacro">
@@ -69,5 +72,5 @@
           <mesh filename="${meshfile}"/>
         </geometry>
-        <material name="light_black"/>
+       <!-- <material name="light_black"/> -->
       </visual>
     </link>
@@ -75,7 +78,7 @@
  <xacro:macro name="create_noa" params="name origin_rpy origin_xyz parent">
   <link name="${name}">
-    <visual>
+   <!-- <visual>
         <origin rpy="0 0 0" xyz="0 0 0"/>
-    </visual>
+    </visual> -->
   </link>
   <joint name="Tool_${name}" type="fixed">

File: urdf/robot_parameters.xacro (robot description, xacro)
@@ -6,8 +6,11 @@
   LABORATORIO / ROBOTICA 2020-1
   PROF: PEDRO CARDENAS
-  ROBOT PROPERTIES - ROBOT DESCRITION
-  AUTHOR: JURGEN KREJCI MUNOZ
+  URDF ROBOT DESCRIPTION EXAMPLE FOR GAZEBO SIMULATION
+  AUTHOR: JURGEN H. KREJCI MUNOZ
+  ROBOT: 2R
   MAIL: jhkrejcim@unal.edu.co
   VERSION: 1.0
+  TESTED ON ROS NOETIC (UBUNTU 20.04.1 LTS)
+  https://github.com/JurgenHK/2R-Manipulator-URDF
   -->
 <robot xmlns:xacro="http://www.ros.org/wiki/xacro">

Commit message: Fixed model scale, corrected controller interface

File: urdf/2r_description.xacro (robot description, xacro)
@@ -3,5 +3,4 @@
   UNIVERSIDAD NACIONAL DE COLOMBIA
   DEPARTAMENTO DE ING. MECANICA Y MECATRONICA
-  SEMILLERO DE ROBOTICA MOMENTUN
   LABORATORIO / ROBOTICA 2020-1
   PROF: PEDRO CARDENAS
@@ -23,5 +22,5 @@
     origin_xyz="0 0 0"
     origin_rpy="0 0 0"
-    meshfile="package://basic_2r_gazebo/CAD/Base.dae"
+    meshfile="package://basic_2r_gazebo/meshes/Base.stl"
     mass="0.00272"
     ixx="0.00000006" ixy="0" ixz="0"
@@ -32,12 +31,12 @@
     type="revolute"
     axis_xyz="0 0 1"
-    origin_rpy="1.57 -1.57 0" origin_xyz="0 2 8.5"
+    origin_rpy="1.57 -1.57 0" origin_xyz="0 0 0.85"
     parent="${link_00_name}" child="${link_01_name}"
     limit_e="100" limit_l="-3.14" limit_u="3.14" limit_v="0.5"
   />
   <xacro:m_link_mesh name="${link_01_name}"
-    origin_xyz="0 0 0"
+    origin_xyz="0 0 -0.2"
     origin_rpy="0 0 0"
-    meshfile="package://basic_2r_gazebo/CAD/Link1.dae"
+    meshfile="package://basic_2r_gazebo/meshes/Link1.stl"
     mass="0.002268"
     ixx="0.0000000181" ixy="0" ixz="0"
@@ -48,12 +47,12 @@
     type="revolute"
     axis_xyz="0 0 1"
-    origin_rpy="0 0 0" origin_xyz="15 0 1"
+    origin_rpy="0 0 0" origin_xyz="1.5 0 0"
     parent="${link_01_name}" child="${link_02_name}"
     limit_e="100" limit_l="-3.14" limit_u="3.14" limit_v="0.5"
   />
   <xacro:m_link_mesh name="${link_02_name}"
-    origin_xyz="0 0 0"
+    origin_xyz="0 0 -0.1"
     origin_rpy="0 0 0"
-    meshfile="package://basic_2r_gazebo/CAD/Link2.dae"
+    meshfile="package://basic_2r_gazebo/meshes/Link2.stl"
     mass="0.002268"
     ixx="0.0000000181" ixy="0" ixz="0"
@@ -64,12 +63,12 @@
     type="prismatic"
     axis_xyz="0 0 1"
-    origin_rpy="0 1.57 -1.57" origin_xyz="15.25 5 1"
+    origin_rpy="0 1.57 -1.57" origin_xyz="1.525 0.5 0"
     parent="${link_02_name}" child="${link_03_name}"
-    limit_e="100" limit_l="0" limit_u="2" limit_v="0.5"
+    limit_e="100" limit_l="0" limit_u="0.2" limit_v="0.5"
   />
   <xacro:m_link_mesh name="${link_03_name}"
     origin_xyz="0 0 0"
     origin_rpy="0 0 0"
-    meshfile="package://basic_2r_gazebo/CAD/Finger.dae"
+    meshfile="package://basic_2r_gazebo/meshes/Finger.stl"
     mass="0.002268"
     ixx="0.0000000181" ixy="0" ixz="0"
@@ -80,7 +79,7 @@
     type="prismatic"
     axis_xyz="0 0 1"
-    origin_rpy="0 -1.57 -1.57" origin_xyz="15.25 -5 1"
+    origin_rpy="0 -1.57 -1.57" origin_xyz="1.525 -0.5 0"
     parent="${link_02_name}" child="${link_04_name}"
-    limit_e="100" limit_l="0" limit_u="2" limit_v="0.5"
+    limit_e="100" limit_l="0" limit_u="0.2" limit_v="0.5"
     mimic_joint="${joint_03_name}" m_multiplier="1" m_offset="0"
   />
@@ -88,5 +87,5 @@
     origin_xyz="0 0 0"
     origin_rpy="0 0 0"
-    meshfile="package://basic_2r_gazebo/CAD/Finger.dae"
+    meshfile="package://basic_2r_gazebo/meshes/Finger.stl"
     mass="0.002268"
     ixx="0.0000000181" ixy="0" ixz="0"
@@ -95,5 +94,5 @@
   />
   <xacro:create_noa name="NOA"
-    origin_xyz="20 0 0"
+    origin_xyz="2 0 0"
     origin_rpy="-1.57 0 -1.57"
     parent="${link_02_name}"

File: urdf/2r_description_gazebo.xacro (robot description, xacro)
@@ -3,5 +3,4 @@
   UNIVERSIDAD NACIONAL DE COLOMBIA
   DEPARTAMENTO DE ING. MECANICA Y MECATRONICA
-  SEMILLERO DE ROBOTICA MOMENTUN
   LABORATORIO / ROBOTICA 2020-1
   PROF: PEDRO CARDENAS
@@ -16,6 +15,6 @@
 <robot name="2R" xmlns:xacro="http://www.ros.org/wiki/xacro">
   <!-- Include-->
-  <xacro:include filename="$(find basic_basic_2r_gazebo)/urdf/links_joints.xacro" />
-  <xacro:include filename="$(find basic_basic_2r_gazebo)/urdf/robot_parameters.xacro" />
+  <xacro:include filename="$(find basic_2r_gazebo)/urdf/links_joints.xacro" />
+  <xacro:include filename="$(find basic_2r_gazebo)/urdf/robot_parameters.xacro" />
   <!-- END - Include -->
   <!-- Robot description -->
@@ -28,64 +27,64 @@
     origin_xyz="0 0 0"
     origin_rpy="0 0 0"
-    meshfile="package://basic_2r_gazebo/CAD/Base.stl"
-    mass="1.024"
-    ixx="170.0" ixy="0" ixz="0"
-    iyy="170.0" iyz="0"
-    izz="170.0"
+    meshfile="package://basic_2r_gazebo/meshes/Base.stl"
+    mass="1"
+    ixx="0.01" ixy="0" ixz="0"
+    iyy="0.01" iyz="0"
+    izz="0.01"
   />
   <xacro:m_joint name="${joint_01_name}"
     type="revolute"
     axis_xyz="0 0 1"
-    origin_rpy="1.57 -1.57 0" origin_xyz="0 2 8.5"
+    origin_rpy="1.57 -1.57 0" origin_xyz="0 0 0.85"
     parent="${link_00_name}" child="${link_01_name}"
-    limit_e="100" limit_l="-3.14" limit_u="3.14" limit_v="0.5"
+    limit_e="10" limit_l="-3.14" limit_u="3.14" limit_v="5.0"
   />
   <xacro:m_link_mesh name="${link_01_name}"
-    origin_xyz="0 0 0"
+    origin_xyz="0 0 -0.2"
     origin_rpy="0 0 0"
-    meshfile="package://basic_2r_gazebo/CAD/Link1.stl"
-    mass="1.570"
-    ixx="130.0" ixy="0" ixz="0"
-    iyy="130.0" iyz="0"
-    izz="90.0"
+    meshfile="package://basic_2r_gazebo/meshes/Link1.stl"
+    mass="1"
+    ixx="0.01" ixy="0" ixz="0"
+    iyy="0.01" iyz="0"
+    izz="0.01"
   />
   <xacro:m_joint name="${joint_02_name}"
     type="revolute"
     axis_xyz="0 0 1"
-    origin_rpy="0 0 0" origin_xyz="15 0 1"
+    origin_rpy="0 0 0" origin_xyz="1.5 0 0"
     parent="${link_01_name}" child="${link_02_name}"
-    limit_e="100" limit_l="-3.14" limit_u="3.14" limit_v="0.5"
+    limit_e="10" limit_l="-3.14" limit_u="3.14" limit_v="5.0"
   />
   <xacro:m_link_mesh name="${link_02_name}"
-    origin_xyz="0 0 0"
+    origin_xyz="0 0 -0.1"
     origin_rpy="0 0 0"
-    meshfile="package://basic_2r_gazebo/CAD/Link2.stl"
-    mass="0.057"
-    ixx="12.0" ixy="0" ixz="0"
-    iyy="12.0" iyz="0"
-    izz="12.0"
+    meshfile="package://basic_2r_gazebo/meshes/Link2.stl"
+    mass="1"
+    ixx="0.01" ixy="0" ixz="0"
+    iyy="0.01" iyz="0"
+    izz="0.01"
   />
   <xacro:m_joint name="${joint_03_name}"
     type="prismatic"
     axis_xyz="0 0 1"
-    origin_rpy="0 1.57 -1.57" origin_xyz="15.25 5 1"
+    origin_rpy="0 1.57 -1.57" origin_xyz="1.525 0.5 0"
     parent="${link_02_name}" child="${link_03_name}"
-    limit_e="100" limit_l="0" limit_u="2" limit_v="0.5"
+    limit_e="10" limit_l="0" limit_u="0.2" limit_v="5.0"
   />
   <xacro:m_link_mesh name="${link_03_name}"
     origin_xyz="0 0 0"
     origin_rpy="0 0 0"
-    meshfile="package://basic_2r_gazebo/CAD/Finger.stl"
-    mass="0.018"
-    ixx="0.5" ixy="0" ixz="0"
-    iyy="0.5" iyz="0"
-    izz="0.5"
+    meshfile="package://basic_2r_gazebo/meshes/Finger.stl"
+    mass="0.5"
+    ixx="0.01" ixy="0" ixz="0"
+    iyy="0.01" iyz="0"
+    izz="0.01"
   />
   <xacro:m_joint_mimic name="${joint_04_name}"
     type="prismatic"
     axis_xyz="0 0 1"
-    origin_rpy="0 -1.57 -1.57" origin_xyz="15.25 -5 1"
+    origin_rpy="0 -1.57 -1.57" origin_xyz="1.525 -0.5 0"
     parent="${link_02_name}" child="${link_04_name}"
-    limit_e="100" limit_l="0" limit_u="2" limit_v="0.5"
+    limit_e="10" limit_l="0" limit_u="0.2" limit_v="5.0"
     mimic_joint="${joint_03_name}" m_multiplier="1" m_offset="0"
   />
@@ -93,9 +92,9 @@
     origin_xyz="0 0 0"
     origin_rpy="0 0 0"
-    meshfile="package://basic_2r_gazebo/CAD/Finger.stl"
-    mass="0.018"
-    ixx="0.5" ixy="0" ixz="0"
-    iyy="0.5" iyz="0"
-    izz="0.5"
+    meshfile="package://basic_2r_gazebo/meshes/Finger.stl"
+    mass="0.5"
+    ixx="0.01" ixy="0" ixz="0"
+    iyy="0.01" iyz="0"
+    izz="0.01"
   />
   <!-- END - Robot description -->

File: urdf/links_joints.xacro (robot description, xacro)
@@ -4,5 +4,4 @@
   DEPARTAMENTO DE ING. MECANICA Y MECATRONICA
   SEMILLERO DE ROBOTICA MOMENTUN
-  LABORATORIO / ROBOTICA 2020-1
   PROF: PEDRO CARDENAS
   URDF ROBOT DESCRIPTION EXAMPLE FOR GAZEBO SIMULATION
@@ -26,8 +25,8 @@
 	      <type>transmission_interface/SimpleTransmission</type>
 	      <joint name="${name}">
-		<hardwareInterface>hardware_interface/EffortJointInterface</hardwareInterface>
+		<hardwareInterface>hardware_interface/PositionJointInterface</hardwareInterface>
 	      </joint>
 	      <actuator name="motor_${name}">
-		<hardwareInterface>hardware_interface/EffortJointInterface</hardwareInterface>
+		<hardwareInterface>hardware_interface/PositionJointInterface</hardwareInterface>
 		<mechanicalReduction>1</mechanicalReduction>
 	      </actuator>
@@ -46,8 +45,8 @@
       <type>transmission_interface/SimpleTransmission</type>
       <joint name="${name}">
-  <hardwareInterface>hardware_interface/EffortJointInterface</hardwareInterface>
+  <hardwareInterface>hardware_interface/PositionJointInterface</hardwareInterface>
       </joint>
       <actuator name="motor_${name}">
-  <hardwareInterface>hardware_interface/EffortJointInterface</hardwareInterface>
+  <hardwareInterface>hardware_interface/PositionJointInterface</hardwareInterface>
   <mechanicalReduction>1</mechanicalReduction>
       </actuator>
@@ -64,5 +63,5 @@
         <origin rpy="${origin_rpy}" xyz="${origin_xyz}" />
         <geometry>
-          <mesh filename="${meshfile}"/>
+          <mesh filename="${meshfile}" scale="0.1 0.1 0.1"/>
         </geometry>
       </collision>
@@ -70,9 +69,14 @@
         <origin rpy="${origin_rpy}" xyz="${origin_xyz}" />
         <geometry>
-          <mesh filename="${meshfile}"/>
+          <mesh filename="${meshfile}" scale="0.1 0.1 0.1"/>
         </geometry>
-       <!-- <material name="light_black"/> -->
+        <material name="Cyan">
+          <color rgba="0 1.0 1.0 1.0"/>
+        </material>
       </visual>
     </link>
+    <gazebo reference="${name}">
+        <material>Gazebo/BlueGlow</material>
+    </gazebo>
  </xacro:macro>
  <xacro:macro name="create_noa" params="name origin_rpy origin_xyz parent">

File: urdf/robot_parameters.xacro (robot description, xacro)
@@ -3,5 +3,4 @@
   UNIVERSIDAD NACIONAL DE COLOMBIA
   DEPARTAMENTO DE ING. MECANICA Y MECATRONICA
-  SEMILLERO DE ROBOTICA MOMENTUN
   LABORATORIO / ROBOTICA 2020-1
   PROF: PEDRO CARDENAS

Commit message: Corrected launch names, updated package info

File: urdf/2r_description.xacro (robot description, xacro)
@@ -9,5 +9,5 @@
   ROBOT: 2R
   MAIL: jhkrejcim@unal.edu.co
-  VERSION: 1.0
+  VERSION: 1.1
   TESTED ON ROS NOETIC (UBUNTU 20.04.1 LTS)
   https://github.com/JurgenHK/2R-Manipulator-URDF
@@ -19,4 +19,11 @@
   <!-- END - Include -->
   <!-- Robot description -->
+  <link name="base_link">
+  </link>
+  <joint name="joint_name" type="fixed">
+    <parent link="base_link"/>
+    <child link="${link_00_name}"/>
+    <origin xyz="0.0 0.0 0.0" rpy="0.0 0.0 0.0"/>
+  </joint>
   <xacro:m_link_mesh name="${link_00_name}"
     origin_xyz="0 0 0"

File: urdf/2r_description_gazebo.xacro (robot description, xacro)
@@ -9,5 +9,5 @@
   ROBOT: 2R
   MAIL: jhkrejcim@unal.edu.co
-  VERSION: 1.0
+  VERSION: 1.1
   TESTED ON ROS NOETIC (UBUNTU 20.04.1 LTS)
   https://github.com/JurgenHK/2R-Manipulator-URDF

File: urdf/links_joints.xacro (robot description, xacro)
@@ -3,5 +3,4 @@
   UNIVERSIDAD NACIONAL DE COLOMBIA
   DEPARTAMENTO DE ING. MECANICA Y MECATRONICA
-  SEMILLERO DE ROBOTICA MOMENTUN
   PROF: PEDRO CARDENAS
   URDF ROBOT DESCRIPTION EXAMPLE FOR GAZEBO SIMULATION
@@ -9,5 +8,5 @@
   ROBOT: 2R
   MAIL: jhkrejcim@unal.edu.co
-  VERSION: 1.0
+  VERSION: 1.1
   TESTED ON ROS NOETIC (UBUNTU 20.04.1 LTS)
   https://github.com/JurgenHK/2R-Manipulator-URDF

File: urdf/robot_parameters.xacro (robot description, xacro)
@@ -9,10 +9,10 @@
   ROBOT: 2R
   MAIL: jhkrejcim@unal.edu.co
-  VERSION: 1.0
+  VERSION: 1.1
   TESTED ON ROS NOETIC (UBUNTU 20.04.1 LTS)
   https://github.com/JurgenHK/2R-Manipulator-URDF
   -->
 <robot xmlns:xacro="http://www.ros.org/wiki/xacro">
-  <xacro:property name="link_00_name" value="base_link" />
+  <xacro:property name="link_00_name" value="robot_base" />
   <xacro:property name="link_01_name" value="link_01" />
   <xacro:property name="link_02_name" value="link_02" />
